File: Additional_Player_PCB.kicad_pcb (KiCad board)
At the start: 2 copper layers, 230 x 119 mm, 14 parts, among them J1 Conn_01x10, SW1 CherryMX, SW2 CherryMX, SW3 CherryMX, SW4 CherryMX, SW5 CherryMX, SW6 CherryMX, SW7 CherryMX, SW8 CherryMX, SW9 CherryMX

Commit message: oops all libraries
Whats a fella gotta do to have pretty 3D models on his board?
Parts:
- J1: footprint Connector_PinHeader_1.00mm:PinHeader_2x05_P1.00mm_Vertical -> Library:PinHeader_2x05_P1.00mm_Vertical
- MH (x4): footprint MountingHole:MountingHole_3.2mm_M3 -> Library:MountingHole_3.2mm_M3
- SW1, SW2, SW3, SW4, SW5, SW6, SW7, SW8, SW9: footprint Button_Switch_Keyboard:SW_Cherry_MX_1.00u_PCB -> Library:SW_Cherry_MX_1.00u_PCB

Commit message: Net Names Added
Didn't realize that annotations didn't function as official net names. Fixed now.
Connections:
- net Net-(J1-Pad1) renamed /START
- net Net-(J1-Pad10) renamed /GND
- net Net-(J1-Pad2) renamed /LEFT
- net Net-(J1-Pad3) renamed /B4
- net Net-(J1-Pad4) renamed /DOWN
- net Net-(J1-Pad5) renamed /B3
- net Net-(J1-Pad6) renamed /RIGHT
- net Net-(J1-Pad7) renamed /B2
- net Net-(J1-Pad8) renamed /UP
- net Net-(J1-Pad9) renamed /B1
Changed lines of the file:
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@@
   )
   (net 0 "")
-  (net 1 "Net-(J1-Pad1)")
-  (net 2 "Net-(J1-Pad2)")
-  (net 3 "Net-(J1-Pad3)")
-  (net 4 "Net-(J1-Pad4)")
-  (net 5 "Net-(J1-Pad5)")
-  (net 6 "Net-(J1-Pad6)")
-  (net 7 "Net-(J1-Pad7)")
-  (net 8 "Net-(J1-Pad8)")
-  (net 9 "Net-(J1-Pad9)")
-  (net 10 "Net-(J1-Pad10)")
+  (net 1 "/START")
+  (net 2 "/LEFT")
+  (net 3 "/B4")
+  (net 4 "/DOWN")
+  (net 5 "/B3")
+  (net 6 "/RIGHT")
+  (net 7 "/B2")
+  (net 8 "/UP")
+  (net 9 "/B1")
+  (net 10 "/GND")
   (footprint "Library:MountingHole_3.2mm_M3" (layer "F.Cu")
     (at 252 38)
@@
     (pad "" np_thru_hole circle (at -7.62 5.08) (size 1.7 1.7) (drill 1.7) (layers *.Cu *.Mask))
     (pad "1" thru_hole circle (at 0 0) (size 2.2 2.2) (drill 1.5) (layers *.Cu *.Mask)
-      (net 9 "Net-(J1-Pad9)") (pintype "passive"))
-    (pad "2" thru_hole circle (at -6.35 2.54) (size 2.2 2.2) (drill 1.5) (layers *.Cu *.Mask)
-      (net 10 "Net-(J1-Pad10)") (pintype "passive"))
+      (net 9 "/B1") (pintype "passive"))
+    (pad "2" thru_hole circle (at -6.35 2.54) (size 2.2 2.2) (drill 1.5) (layers *.Cu *.Mask)
+      (net 10 "/GND") (pintype "passive"))
     (model "${KICAD6_3DMODEL_DIR}/Button_Switch_Keyboard.3dshapes/SW_Cherry_MX_1.00u_PCB.wrl" hide
       (offset (xyz 0 0 0))
@@
     (pad "" np_thru_hole circle (at -7.62 5.08) (size 1.7 1.7) (drill 1.7) (layers *.Cu *.Mask))
     (pad "1" thru_hole circle (at 0 0) (size 2.2 2.2) (drill 1.5) (layers *.Cu *.Mask)
-      (net 3 "Net-(J1-Pad3)") (pintype "passive"))
-    (pad "2" thru_hole circle (at -6.35 2.54) (size 2.2 2.2) (drill 1.5) (layers *.Cu *.Mask)
-      (net 10 "Net-(J1-Pad10)") (pintype "passive"))
+      (net 3 "/B4") (pintype "passive"))
+    (pad "2" thru_hole circle (at -6.35 2.54) (size 2.2 2.2) (drill 1.5) (layers *.Cu *.Mask)
+      (net 10 "/GND") (pintype "passive"))
     (model "${KICAD6_3DMODEL_DIR}/Button_Switch_Keyboard.3dshapes/SW_Cherry_MX_1.00u_PCB.wrl" hide
       (offset (xyz 0 0 0))
@@
     (pad "" np_thru_hole circle (at -7.62 5.08) (size 1.7 1.7) (drill 1.7) (layers *.Cu *.Mask))
     (pad "1" thru_hole circle (at 0 0) (size 2.2 2.2) (drill 1.5) (layers *.Cu *.Mask)
-      (net 8 "Net-(J1-Pad8)") (pintype "passive"))
-    (pad "2" thru_hole circle (at -6.35 2.54) (size 2.2 2.2) (drill 1.5) (layers *.Cu *.Mask)
-      (net 10 "Net-(J1-Pad10)") (pintype "passive"))
+      (net 8 "/UP") (pintype "passive"))
+    (pad "2" thru_hole circle (at -6.35 2.54) (size 2.2 2.2) (drill 1.5) (layers *.Cu *.Mask)
+      (net 10 "/GND") (pintype "passive"))
     (model "${KICAD6_3DMODEL_DIR}/Button_Switch_Keyboard.3dshapes/SW_Cherry_MX_1.00u_PCB.wrl" hide
       (offset (xyz 0 0 0))
@@
     (pad "" np_thru_hole circle (at 2.54 5.08) (size 1.7 1.7) (drill 1.7) (layers *.Cu *.Mask))
     (pad "1" thru_hole circle (at 0 0) (size 2.2 2.2) (drill 1.5) (layers *.Cu *.Mask)
-      (net 6 "Net-(J1-Pad6)") (pintype "passive"))
-    (pad "2" thru_hole circle (at -6.35 2.54) (size 2.2 2.2) (drill 1.5) (layers *.Cu *.Mask)
-      (net 10 "Net-(J1-Pad10)") (pintype "passive"))
+      (net 6 "/RIGHT") (pintype "passive"))
+    (pad "2" thru_hole circle (at -6.35 2.54) (size 2.2 2.2) (drill 1.5) (layers *.Cu *.Mask)
+      (net 10 "/GND") (pintype "passive"))
     (model "${KICAD6_3DMODEL_DIR}/Button_Switch_Keyboard.3dshapes/SW_Cherry_MX_1.00u_PCB.wrl" hide
       (offset (xyz 0 0 0))
@@
     (pad "" np_thru_hole circle (at -2.54 5.08) (size 4 4) (drill 4) (layers *.Cu *.Mask))
     (pad "1" thru_hole circle (at 0 0) (size 2.2 2.2) (drill 1.5) (layers *.Cu *.Mask)
-      (net 1 "Net-(J1-Pad1)") (pintype "passive"))
-    (pad "2" thru_hole circle (at -6.35 2.54) (size 2.2 2.2) (drill 1.5) (layers *.Cu *.Mask)
-      (net 10 "Net-(J1-Pad10)") (pintype "passive"))
+      (net 1 "/START") (pintype "passive"))
+    (pad "2" thru_hole circle (at -6.35 2.54) (size 2.2 2.2) (drill 1.5) (layers *.Cu *.Mask)
+      (net 10 "/GND") (pintype "passive"))
     (model "${KICAD6_3DMODEL_DIR}/Button_Switch_Keyboard.3dshapes/SW_Cherry_MX_1.00u_PCB.wrl" hide
       (offset (xyz 0 0 0))
@@
     (pad "" np_thru_hole circle (at -7.62 5.08) (size 1.7 1.7) (drill 1.7) (layers *.Cu *.Mask))
     (pad "1" thru_hole circle (at 0 0) (size 2.2 2.2) (drill 1.5) (layers *.Cu *.Mask)
-      (net 4 "Net-(J1-Pad4)") (pintype "passive"))
-    (pad "2" thru_hole circle (at -6.35 2.54) (size 2.2 2.2) (drill 1.5) (layers *.Cu *.Mask)
-      (net 10 "Net-(J1-Pad10)") (pintype "passive"))
+      (net 4 "/DOWN") (pintype "passive"))
+    (pad "2" thru_hole circle (at -6.35 2.54) (size 2.2 2.2) (drill 1.5) (layers *.Cu *.Mask)
+      (net 10 "/GND") (pintype "passive"))
     (model "${KICAD6_3DMODEL_DIR}/Button_Switch_Keyboard.3dshapes/SW_Cherry_MX_1.00u_PCB.wrl" hide
       (offset (xyz 0 0 0))
@@
     (pad "" np_thru_hole circle (at 2.54 5.08) (size 1.7 1.7) (drill 1.7) (layers *.Cu *.Mask))
     (pad "1" thru_hole circle (at 0 0) (size 2.2 2.2) (drill 1.5) (layers *.Cu *.Mask)
-      (net 2 "Net-(J1-Pad2)") (pintype "passive"))
-    (pad "2" thru_hole circle (at -6.35 2.54) (size 2.2 2.2) (drill 1.5) (layers *.Cu *.Mask)
-      (net 10 "Net-(J1-Pad10)") (pintype "passive"))
+      (net 2 "/LEFT") (pintype "passive"))
+    (pad "2" thru_hole circle (at -6.35 2.54) (size 2.2 2.2) (drill 1.5) (layers *.Cu *.Mask)
+      (net 10 "/GND") (pintype "passive"))
     (model "${KICAD6_3DMODEL_DIR}/Button_Switch_Keyboard.3dshapes/SW_Cherry_MX_1.00u_PCB.wrl" hide
       (offset (xyz 0 0 0))
@@
     (pad "" np_thru_hole circle (at -2.54 5.08) (size 4 4) (drill 4) (layers *.Cu *.Mask))
     (pad "1" thru_hole circle (at 0 0) (size 2.2 2.2) (drill 1.5) (layers *.Cu *.Mask)
-      (net 5 "Net-(J1-Pad5)") (pintype "passive"))
-    (pad "2" thru_hole circle (at -6.35 2.54) (size 2.2 2.2) (drill 1.5) (layers *.Cu *.Mask)
-      (net 10 "Net-(J1-Pad10)") (pintype "passive"))
+      (net 5 "/B3") (pintype "passive"))
+    (pad "2" thru_hole circle (at -6.35 2.54) (size 2.2 2.2) (drill 1.5) (layers *.Cu *.Mask)
+      (net 10 "/GND") (pintype "passive"))
     (model "${KICAD6_3DMODEL_DIR}/Button_Switch_Keyboard.3dshapes/SW_Cherry_MX_1.00u_PCB.wrl" hide
       (offset (xyz 0 0 0))
@@
     (pad "" np_thru_hole circle (at 2.54 5.08) (size 1.7 1.7) (drill 1.7) (layers *.Cu *.Mask))
     (pad "1" thru_hole circle (at 0 0) (size 2.2 2.2) (drill 1.5) (layers *.Cu *.Mask)
-      (net 7 "Net-(J1-Pad7)") (pintype "passive"))
-    (pad "2" thru_hole circle (at -6.35 2.54) (size 2.2 2.2) (drill 1.5) (layers *.Cu *.Mask)
-      (net 10 "Net-(J1-Pad10)") (pintype "passive"))
+      (net 7 "/B2") (pintype "passive"))
+    (pad "2" thru_hole circle (at -6.35 2.54) (size 2.2 2.2) (drill 1.5) (layers *.Cu *.Mask)
+      (net 10 "/GND") (pintype "passive"))
     (model "${KICAD6_3DMODEL_DIR}/Button_Switch_Keyboard.3dshapes/SW_Cherry_MX_1.00u_PCB.wrl" hide
       (offset (xyz 0 0 0))
@@
     (fp_line (start -0.075 0.5) (end 1.65 0.5) (layer "B.Fab") (width 0.1))
     (pad "1" thru_hole rect (at 0 0) (size 0.85 0.85) (drill 0.5) (layers *.Cu *.Mask)
-      (net 1 "Net-(J1-Pad1)") (pinfunction "Pin_1") (pintype "passive"))
+      (net 1 "/START") (pinfunction "Pin_1") (pintype "passive"))
     (pad "2" thru_hole oval (at 1 0) (size 0.85 0.85) (drill 0.5) (layers *.Cu *.Mask)
-      (net 2 "Net-(J1-Pad2)") (pinfunction "Pin_2") (pintype "passive"))
+      (net 2 "/LEFT") (pinfunction "Pin_2") (pintype "passive"))
     (pad "3" thru_hole oval (at 0 -1) (size 0.85 0.85) (drill 0.5) (layers *.Cu *.Mask)
-      (net 3 "Net-(J1-Pad3)") (pinfunction "Pin_3") (pintype "passive"))
+      (net 3 "/B4") (pinfunction "Pin_3") (pintype "passive"))
     (pad "4" thru_hole oval (at 1 -1) (size 0.85 0.85) (drill 0.5) (layers *.Cu *.Mask)
-      (net 4 "Net-(J1-Pad4)") (pinfunction "Pin_4") (pintype "passive"))
+      (net 4 "/DOWN") (pinfunction "Pin_4") (pintype "passive"))
     (pad "5" thru_hole oval (at 0 -2) (size 0.85 0.85) (drill 0.5) (layers *.Cu *.Mask)
-      (net 5 "Net-(J1-Pad5)") (pinfunction "Pin_5") (pintype "passive"))
+      (net 5 "/B3") (pinfunction "Pin_5") (pintype "passive"))
     (pad "6" thru_hole oval (at 1 -2) (size 0.85 0.85) (drill 0.5) (layers *.Cu *.Mask)
-      (net 6 "Net-(J1-Pad6)") (pinfunction "Pin_6") (pintype "passive"))
+      (net 6 "/RIGHT") (pinfunction "Pin_6") (pintype "passive"))
     (pad "7" thru_hole oval (at 0 -3) (size 0.85 0.85) (drill 0.5) (layers *.Cu *.Mask)
-      (net 7 "Net-(J1-Pad7)") (pinfunction "Pin_7") (pintype "passive"))
+      (net 7 "/B2") (pinfunction "Pin_7") (pintype "passive"))
     (pad "8" thru_hole oval (at 1 -3) (size 0.85 0.85) (drill 0.5) (layers *.Cu *.Mask)
-      (net 8 "Net-(J1-Pad8)") (pinfunction "Pin_8") (pintype "passive"))
+      (net 8 "/UP") (pinfunction "Pin_8") (pintype "passive"))
     (pad "9" thru_hole oval (at 0 -4) (size 0.85 0.85) (drill 0.5) (layers *.Cu *.Mask)
-      (net 9 "Net-(J1-Pad9)") (pinfunction "Pin_9") (pintype "passive"))
+      (net 9 "/B1") (pinfunction "Pin_9") (pintype "passive"))
     (pad "10" thru_hole oval (at 1 -4) (size 0.85 0.85) (drill 0.5) (layers *.Cu *.Mask)
-      (net 10 "Net-(J1-Pad10)") (pinfunction "Pin_10") (pintype "passive"))
+      (net 10 "/GND") (pinfunction "Pin_10") (pintype "passive"))
     (model "${KICAD6_3DMODEL_DIR}/Connector_PinHeader_1.00mm.3dshapes/PinHeader_2x05_P1.00mm_Vertical.wrl"
       (offset (xyz 0 0 0))

Commit message: Correct J1 connector
Mil vs. MM, what's the deal?
Parts:
- J1: value Conn_01x10 -> PinHeader_2x05_P2.54mm_Vertical; footprint Library:PinHeader_2x05_P1.00mm_Vertical -> Connector_PinHeader_2.54mm:PinHeader_2x05_P2.54mm_Vertical
- moved J1 14.5 mm to (76.6, 38.1)
Connections:
- net /GND renamed GND
Routing:
- net GND: track 357.8 -> 0.00 mm
- net /LEFT: track 57.9 -> 75.7 mm
- net /START: track 87.7 -> 72.0 mm
- net /B4: track 192.1 -> 179.4 mm
- net /DOWN: track 89.3 -> 100.2 mm
- net /B2: track 143.0 -> 133.3 mm
- net /UP: track 33.4 -> 41.0 mm
- net /B1: track 129.0 -> 121.9 mm
- net /B3: track 167.6 -> 161.6 mm
- net /RIGHT: track 92.5 -> 98.4 mm
- added copper zone on B.Cu, net GND
Other:
- board text added: "1"
- board text added: "B1"
- board text added: "B2"
- board text added: "B3"
- board text added: "B4"
- board text added: "Down"
- board text added: "Left"
- board text added: "Right"
- board text added: "Start"
- board text added: "Up"
- board text added: "haha stinky"
